Commit message: backup: save current workspace state

File: sim/robot/robot.urdf (robot description, URDF)
Before this commit: robot robot, 9 links, 8 joints
Joints:
- joint base_link_旋转-3: axis -0.002609 -0.9999869999999998 0.004304000000000168 -> -0.0026091176 -0.9999873332 0.0043041762
- joint link1_right_旋转-5: axis -0.002609 -0.999987 0.0043040000000000005 -> 0.0026091176 0.9999873332 -0.0043041762
- joint link2_left_旋转-13: axis 0.0026090000000001112 0.999987 -0.004304 -> -0.0026090000000001112 -0.999987 0.004304

File: sim/robot/robot_yup_backup.urdf (robot description, URDF)
Before this commit: robot robot, 9 links, 8 joints
Joints:
- joint base_link_旋转-3: axis -0.002609 -0.9999869999999998 0.004304000000000168 -> 0.002609 0.9999869999999998 -0.004304000000000168
- joint link2_left_旋转-13: axis 0.0026090000000001112 0.999987 -0.004304 -> -0.0026090000000001112 -0.999987 0.004304

Commit message: chore: backup before coordinate model rework

File: sim/robot/robot.urdf (robot description, URDF)
Before this commit: robot robot, 9 links, 8 joints
Joints:
- joint base_link_旋转-1: axis 0.002609 -0.9999869999999998 0.004304000000000139 -> -0.0026091176 -0.9999873332 0.0043041762
- joint base_link_旋转-3: axis -0.0026091176 -0.9999873332 0.0043041762 -> 0.002609 -0.9999869999999998 0.004304000000000139
- joint link1_right_旋转-5: origin xyz=-0.06746535000000002 -0.015289760000000001 -0.026379890000000027 rpy=3.141592653589793 0.0 0.0 -> xyz=-0.06746535000000002 -0.015289760000000001 -0.026379890000000027 rpy=0 0 0
- joint link2_right_旋转-12: origin xyz=0.07559893 7.8990000000001e-05 0.06417946999999999 rpy=2.0293072715139053e-17 0.0 0.0 -> xyz=0.075598929999999995 -7.8990000000001004e-05 -0.064179469999999988 rpy=-3.1415926535897931 -0 0

Commit message: backup

File: sim/robot/robot.urdf (robot description, URDF)
Before this commit: robot robot, 9 links, 8 joints
Links:
- link link2_right: mass 0.4808903080599056 -> 0.4808903080599057
Joints:
- joint base_link_旋转-1: axis -0.0026091176 -0.9999873332 0.0043041762 -> 0.002609 -0.9999869999999998 0.004304000000000125
- joint base_link_旋转-3: axis 0.002609 -0.9999869999999998 0.004304000000000139 -> 0.002609 0.9999869999999998 -0.004304000000000139
- joint link1_right_旋转-5: axis 0.0026091176 0.9999873332 -0.0043041762 -> -0.002609 0.999987 -0.004304

Commit message: backup: pre-refactor snapshot of LQR/VMC/Phase controllers
Saves current state of jump/balance controller patches (C1 wheel_vel
threshold, CROUCH integral reset, flight pre-tuck, lowered extend
feedforward) before architectural cleanup that drops wheel_pos from LQR
state and removes the cascading patches it requires.

File: sim/robot/robot.urdf (robot description, URDF)
Before this commit: robot robot, 9 links, 8 joints
Links:
- link base_link: mass 6.714653948788012 -> 0.94
- link link1_left: mass 0.2530518137091047 -> 0.04
- link link1_right: mass 0.2530518137091047 -> 0.04
- link link2_left: mass 0.4808903080599057 -> 0.08
- link link2_right: mass 0.4808903080599057 -> 0.08
- link link3_left: mass 0.07190706335416745 -> 0.01
- link link3_right: mass 0.07190706335416698 -> 0.01
- link wheel_left: mass 0.9552209288691303 -> 0.50
- link wheel_right: mass 0.9552209288691303 -> 0.50

Commit message: update

File: sim/robot/robot.urdf (robot description, URDF)
Before this commit: robot robot, 9 links, 8 joints
Joints:
- joint base_link_旋转-1: limit lower=0.261799 upper=1.658063 effort=1000000 velocity=1000000 -> lower=-0.110000 upper=1.658063 effort=1000000 velocity=1000000
- joint base_link_旋转-2: limit lower=0.261799 upper=1.658063 effort=1000000 velocity=1000000 -> lower=-0.110000 upper=1.658063 effort=1000000 velocity=1000000

Commit message: feat(jump): rebuild jump pipeline — 9-10cm hop with controlled drift
- New ConstantAccelerationTrajectory for EXTEND: derives duration from
  stroke + v_takeoff so motor pushes at constant a from t=0 instead of
  QuarticTrajectory's late-burst profile that couldn't lift body in time.
- VMC EXTEND: after t > duration, set kp_motor=0 (keep ff_torque + kd).
  Stale h_target clipping was making PID pull body back to ground while
  motor over-extended past h_high — vz dropped 1.5→0.5 m/s in 2ms.
- VMC FLIGHT: leg motors apply symmetric -Kd*pitch_rate torque using
  Newton-3rd reaction to damp body pitch_rate in flight (no contact, so
  legs act as reaction wheels). Without this pitch_rate accumulated to
  -6 rad/s during EXTEND, flipping body in 250ms airborne.
- Combined controller FLIGHT branch forwards VMC output (previously
  returned zeros, killing the new damping).
- Phase machine: EXTEND→FLIGHT requires sustained ncon=0 (>=5ms) plus
  vz>0.3 to ignore bouncing transients; 2x duration safety timeout.
- LQR target during jump phases drops pitch_lean (was treating extend
  wheel-velocity transient as 'should lean forward'); pure equilibrium
  pitch + wheel_vel=0.
- launch_mujoco._trigger_jump_on_rising_edge: cmd_jump slider now acts
  as a button (any >0.01 → amp=1.0). MuJoCo Control sliders are hard to
  drag to 1.0 — partial values produced 22mm jumps.
- air_height_max=0.40 default: ~94mm jump with ~3cm drift. 0.50 gives
  113mm but 33cm drift (LQR pitch recovery during LAND drives wheels).
- Added scripts/verify_jump_height.py + diagnostic [jump-trigger] log.
- All 82 tests pass.

File: sim/robot/robot.urdf (robot description, URDF)
Before this commit: robot robot, 9 links, 8 joints
Joints:
- joint base_link_旋转-1: limit lower=-0.110000 upper=1.658063 effort=1000000 velocity=1000000 -> lower=-0.110000 upper=0.600000 effort=1000000 velocity=1000000
- joint base_link_旋转-2: limit lower=-0.110000 upper=1.658063 effort=1000000 velocity=1000000 -> lower=-0.110000 upper=0.600000 effort=1000000 velocity=1000000
